File: eagle-schematics/joystick-tester-smd.brd (EAGLE design)
At the start: 22.9 x 63.5 mm, 13 parts

Commit message: Updated battery layout
Parts:
- removed U$1: CR2032-SMD_2PX30MM, Per:CR2032_2P30_SMD
- added BT1: CR2032, Per:CR2032_2P30SMD_20MM_COMBO
- R1, R2, R3, R4, R5: value 180R -> 220R
- X2: value (none) -> DB9
- renumbered D7 to D5, R7 to R5
Connections:
- net GND: now also BT1.P$2, BT1.P$4; no longer U$1.P$2
- net VCC: now also BT1.P$1, BT1.P$3; no longer U$1.P$1
Routing:
- net VCC: track 76.8 -> 80.9 mm
Changed lines of the file:
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@@
 <layer number="25" name="tNames" color="7" fill="1" visible="yes" active="yes"/>
 <layer number="26" name="bNames" color="7" fill="1" visible="yes" active="yes"/>
-<layer number="27" name="tValues" color="7" fill="1" visible="yes" active="yes"/>
+<layer number="27" name="tValues" color="7" fill="1" visible="no" active="yes"/>
 <layer number="28" name="bValues" color="7" fill="1" visible="yes" active="yes"/>
 <layer number="29" name="tStop" color="7" fill="3" visible="no" active="yes"/>
@@
 <attribute name="VALUE" x="21.185" y="21.971" size="1.27" layer="21" ratio="10" rot="R180"/>
 </element>
-<element name="D7" library="SparkFun-LED" package="LED-1206" value="Fire" x="11.66" y="19.05" smashed="yes" rot="R180">
+<element name="D5" library="SparkFun-LED" package="LED-1206" value="Fire" x="11.66" y="19.05" smashed="yes" rot="R180">
 <attribute name="NAME" x="8.128" y="19.788" size="0.889" layer="25" ratio="10" rot="R270"/>
 <attribute name="VALUE" x="13.565" y="21.971" size="1.27" layer="21" ratio="10" rot="R180"/>
 </element>
-<element name="R1" library="rcl" library_urn="urn:adsk.eagle:library:334" package="M0805" package3d_urn="urn:adsk.eagle:package:23556/2" value="180R" x="11.684" y="24.13" smashed="yes">
+<element name="R1" library="rcl" library_urn="urn:adsk.eagle:library:334" package="M0805" package3d_urn="urn:adsk.eagle:package:23556/2" value="220R" x="11.684" y="24.13" smashed="yes">
 <attribute name="NAME" x="8.636" y="24.892" size="0.889" layer="25" rot="R270"/>
 <attribute name="POPULARITY" value="45" x="11.684" y="24.13" size="1.778" layer="27" display="off"/>
@@
 <attribute name="VALUE" x="10.414" y="21.59" size="1.27" layer="27"/>
 </element>
-<element name="R2" library="rcl" library_urn="urn:adsk.eagle:library:334" package="M0805" package3d_urn="urn:adsk.eagle:package:23556/2" value="180R" x="11.43" y="8.89" smashed="yes">
+<element name="R2" library="rcl" library_urn="urn:adsk.eagle:library:334" package="M0805" package3d_urn="urn:adsk.eagle:package:23556/2" value="220R" x="11.43" y="8.89" smashed="yes">
 <attribute name="NAME" x="8.382" y="9.652" size="0.889" layer="25" rot="R270"/>
 <attribute name="POPULARITY" value="45" x="11.43" y="8.89" size="1.778" layer="27" display="off"/>
@@
 <attribute name="VALUE" x="12.319" y="6.731" size="1.27" layer="27"/>
 </element>
-<element name="R3" library="rcl" library_urn="urn:adsk.eagle:library:334" package="M0805" package3d_urn="urn:adsk.eagle:package:23556/2" value="180R" x="4.445" y="16.51" smashed="yes">
+<element name="R3" library="rcl" library_urn="urn:adsk.eagle:library:334" package="M0805" package3d_urn="urn:adsk.eagle:package:23556/2" value="220R" x="4.445" y="16.51" smashed="yes">
 <attribute name="NAME" x="1.397" y="17.272" size="0.889" layer="25" rot="R270"/>
 <attribute name="POPULARITY" value="45" x="4.445" y="16.51" size="1.778" layer="27" display="off"/>
@@
 <attribute name="VALUE" x="8.255" y="14.097" size="1.27" layer="27" rot="R180"/>
 </element>
-<element name="R4" library="rcl" library_urn="urn:adsk.eagle:library:334" package="M0805" package3d_urn="urn:adsk.eagle:package:23556/2" value="180R" x="19.05" y="16.51" smashed="yes">
+<element name="R4" library="rcl" library_urn="urn:adsk.eagle:library:334" package="M0805" package3d_urn="urn:adsk.eagle:package:23556/2" value="220R" x="19.05" y="16.51" smashed="yes">
 <attribute name="NAME" x="16.002" y="17.272" size="0.889" layer="25" rot="R270"/>
 <attribute name="POPULARITY" value="45" x="19.05" y="16.51" size="1.778" layer="27" display="off"/>
@@
 <attribute name="VALUE" x="22.86" y="13.843" size="1.27" layer="27" rot="R180"/>
 </element>
-<element name="R7" library="rcl" library_urn="urn:adsk.eagle:library:334" package="M0805" package3d_urn="urn:adsk.eagle:package:23556/2" value="180R" x="11.684" y="16.51" smashed="yes" rot="R180">
+<element name="R5" library="rcl" library_urn="urn:adsk.eagle:library:334" package="M0805" package3d_urn="urn:adsk.eagle:package:23556/2" value="220R" x="11.684" y="16.51" smashed="yes" rot="R180">
 <attribute name="NAME" x="8.636" y="17.272" size="0.889" layer="25" rot="R270"/>
 <attribute name="POPULARITY" value="45" x="11.684" y="16.51" size="1.778" layer="27" rot="R180" display="off"/>
@@
 <attribute name="VALUE" x="12.954" y="19.05" size="1.27" layer="27" rot="R180"/>
 </element>
-<element name="U$1" library="Per" package="CR2032_2P30_SMD" value="CR2032-SMD_2PX30MM" x="11.557" y="46.863" smashed="yes" rot="R180"/>
-<element name="X2" library="con-subd" library_urn="urn:adsk.eagle:library:189" package="M09D" package3d_urn="urn:adsk.eagle:package:10300/1" value="" x="11.43" y="-3.81" smashed="yes" rot="R180">
+<element name="X2" library="con-subd" library_urn="urn:adsk.eagle:library:189" package="M09D" package3d_urn="urn:adsk.eagle:package:10300/1" value="DB9" x="11.43" y="-3.81" smashed="yes" rot="R180">
 <attribute name="MF" value="" x="-19.05" y="33.02" size="1.778" layer="27" rot="R180" display="off"/>
 <attribute name="MPN" value="" x="-19.05" y="33.02" size="1.778" layer="27" rot="R180" display="off"/>
@@
 <attribute name="OC_FARNELL" value="unknown" x="-19.05" y="33.02" size="1.778" layer="27" rot="R180" display="off"/>
 <attribute name="OC_NEWARK" value="unknown" x="-19.05" y="33.02" size="1.778" layer="27" rot="R180" display="off"/>
-<attribute name="VALUE" x="10.16" y="6.35" size="1.778" layer="27" ratio="10" rot="R180"/>
+<attribute name="VALUE" x="1.27" y="-7.62" size="1.778" layer="27" ratio="10" rot="R180"/>
 </element>
 <element name="U$2" library="oshw" package="OSHW_8MM" value="" x="10.16" y="17.145" smashed="yes" rot="MR90"/>
+<element name="BT1" library="Per" package="CR2032_2P30SMD_20MM_COMBO" value="CR2032" x="11.43" y="46.736" smashed="yes" rot="R180">
+<attribute name="NAME" x="12.7" y="42.926" size="1.27" layer="21" rot="R180"/>
+<attribute name="VALUE" x="13.97" y="51.816" size="1.016" layer="25" rot="R180"/>
+</element>
 </elements>
 <signals>
@@
 <signal name="GND">
 <contactref element="X2" pad="8"/>
-<contactref element="U$1" pad="P$2"/>
 <polygon width="0.1" layer="1" rank="3">
 <vertex x="-1.27" y="-1.27"/>
@@
 <wire x1="15.24" y1="17.78" x2="15.24" y2="16.4084" width="0.1524" layer="16"/>
 <wire x1="12.8016" y1="13.97" x2="12.8016" y2="2.2352" width="0.1524" layer="16"/>
+<contactref element="BT1" pad="P$2"/>
+<contactref element="BT1" pad="P$4"/>
 </signal>
 <signal name="FIRE">
-<contactref element="R7" pad="1"/>
+<contactref element="R5" pad="1"/>
 <contactref element="X2" pad="6"/>
 <wire x1="9.4488" y1="13.4112" x2="12.4968" y2="16.4592" width="0.1524" layer="1"/>
@@
 </signal>
 <signal name="N$3">
-<contactref element="R7" pad="2"/>
-<contactref element="D7" pad="C"/>
+<contactref element="R5" pad="2"/>
+<contactref element="D5" pad="C"/>
 <wire x1="10.2108" y1="17.0688" x2="10.2108" y2="19.05" width="0.1524" layer="1"/>
 <wire x1="10.668" y1="16.6116" x2="10.2108" y2="17.0688" width="0.1524" layer="1"/>
@@
 <contactref element="D4" pad="A"/>
 <contactref element="X2" pad="7"/>
-<contactref element="D7" pad="A"/>
-<contactref element="U$1" pad="P$1"/>
+<contactref element="D5" pad="A"/>
 <wire x1="13.2588" y1="15.24" x2="13.2588" y2="11.43" width="0.1524" layer="1"/>
 <wire x1="13.5636" y1="15.5448" x2="13.2588" y2="15.24" width="0.1524" layer="1"/>
@@
 <wire x1="7.62" y1="22.7584" x2="7.62" y2="29.21" width="0.1524" layer="16"/>
 <via x="7.62" y="29.21" extent="1-16" drill="0.35"/>
-<wire x1="7.62" y1="29.21" x2="11.049" y2="32.639" width="0.1524" layer="1"/>
-<wire x1="11.049" y1="32.639" x2="11.557" y2="32.385" width="0.1524" layer="1"/>
+<contactref element="BT1" pad="P$1"/>
+<contactref element="BT1" pad="P$3"/>
+<wire x1="7.62" y1="29.21" x2="10.668" y2="32.258" width="0.1524" layer="1"/>
+<wire x1="10.668" y1="32.258" x2="11.43" y2="32.258" width="0.1524" layer="1"/>
+<wire x1="11.43" y1="36.736" x2="11.43" y2="32.258" width="0.3048" layer="1"/>
 </signal>
 </signals>

Commit message: Update schematics
Parts:
- added U$1: RETRONINJA_TEXT, PCBGraphics:RETRONINJA_TEXT_17MM
- renumbered X2 to X1
Changed lines of the file:
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@@
 <attribute name="VALUE" x="12.954" y="19.05" size="1.27" layer="27" rot="R180"/>
 </element>
-<element name="X2" library="con-subd" library_urn="urn:adsk.eagle:library:189" package="M09D" package3d_urn="urn:adsk.eagle:package:10300/1" value="DB9" x="11.43" y="-3.81" smashed="yes" rot="R180">
+<element name="X1" library="con-subd" library_urn="urn:adsk.eagle:library:189" package="M09D" package3d_urn="urn:adsk.eagle:package:10300/1" value="DB9" x="11.43" y="-3.81" smashed="yes" rot="R180">
 <attribute name="MF" value="" x="-19.05" y="33.02" size="1.778" layer="27" rot="R180" display="off"/>
 <attribute name="MPN" value="" x="-19.05" y="33.02" size="1.778" layer="27" rot="R180" display="off"/>
@@
 <attribute name="VALUE" x="13.97" y="51.816" size="1.016" layer="25" rot="R180"/>
 </element>
+<element name="U$1" library="PCBGraphics" package="RETRONINJA_TEXT_17MM" value="RETRONINJA_TEXT" x="3.81" y="-21.59" smashed="yes"/>
 </elements>
 <signals>
 <signal name="UP">
 <contactref element="R1" pad="2"/>
-<contactref element="X2" pad="1"/>
+<contactref element="X1" pad="1"/>
 <wire x1="12.4968" y1="23.622" x2="12.4968" y2="24.0792" width="0.1524" layer="1"/>
 <wire x1="6.5532" y1="17.6784" x2="12.4968" y2="23.622" width="0.1524" layer="1"/>
@@
 <signal name="DOWN">
 <contactref element="R2" pad="2"/>
-<contactref element="X2" pad="2"/>
+<contactref element="X1" pad="2"/>
 <wire x1="12.3444" y1="6.096" x2="12.3444" y2="8.8392" width="0.1524" layer="1"/>
 <wire x1="8.5344" y1="2.286" x2="12.3444" y2="6.096" width="0.1524" layer="1"/>
@@
 <signal name="LEFT">
 <contactref element="R3" pad="2"/>
-<contactref element="X2" pad="3"/>
+<contactref element="X1" pad="3"/>
 <wire x1="9.4488" y1="12.4968" x2="5.4864" y2="16.4592" width="0.1524" layer="1"/>
 <wire x1="10.8204" y1="12.4968" x2="9.4488" y2="12.4968" width="0.1524" layer="1"/>
@@
 <signal name="RIGHT">
 <contactref element="R4" pad="2"/>
-<contactref element="X2" pad="4"/>
+<contactref element="X1" pad="4"/>
 <wire x1="19.9644" y1="8.2296" x2="19.9644" y2="16.4592" width="0.1524" layer="1"/>
 <wire x1="14.3256" y1="2.5908" x2="19.9644" y2="8.2296" width="0.1524" layer="1"/>
@@
 </signal>
 <signal name="GND">
-<contactref element="X2" pad="8"/>
+<contactref element="X1" pad="8"/>
 <polygon width="0.1" layer="1" rank="3">
 <vertex x="-1.27" y="-1.27"/>
@@
 <signal name="FIRE">
 <contactref element="R5" pad="1"/>
-<contactref element="X2" pad="6"/>
+<contactref element="X1" pad="6"/>
 <wire x1="9.4488" y1="13.4112" x2="12.4968" y2="16.4592" width="0.1524" layer="1"/>
 <wire x1="9.4488" y1="4.572" x2="9.4488" y2="13.4112" width="0.1524" layer="16"/>
@@
 <contactref element="D3" pad="A"/>
 <contactref element="D4" pad="A"/>
-<contactref element="X2" pad="7"/>
+<contactref element="X1" pad="7"/>
 <contactref element="D5" pad="A"/>
 <wire x1="13.2588" y1="15.24" x2="13.2588" y2="11.43" width="0.1524" layer="1"/>

Commit message: Update schematics
Parts:
- removed U$1: RETRONINJA_TEXT, PCBGraphics:RETRONINJA_TEXT_17MM
- X1: value DB9 -> DE-9M
Changed lines of the file:
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@@
 <attribute name="VALUE" x="12.954" y="19.05" size="1.27" layer="27" rot="R180"/>
 </element>
-<element name="X1" library="con-subd" library_urn="urn:adsk.eagle:library:189" package="M09D" package3d_urn="urn:adsk.eagle:package:10300/1" value="DB9" x="11.43" y="-3.81" smashed="yes" rot="R180">
+<element name="X1" library="con-subd" library_urn="urn:adsk.eagle:library:189" package="M09D" package3d_urn="urn:adsk.eagle:package:10300/1" value="DE-9M" x="11.43" y="-3.81" smashed="yes" rot="R180">
 <attribute name="MF" value="" x="-19.05" y="33.02" size="1.778" layer="27" rot="R180" display="off"/>
 <attribute name="MPN" value="" x="-19.05" y="33.02" size="1.778" layer="27" rot="R180" display="off"/>
@@
 <attribute name="VALUE" x="13.97" y="51.816" size="1.016" layer="25" rot="R180"/>
 </element>
-<element name="U$1" library="PCBGraphics" package="RETRONINJA_TEXT_17MM" value="RETRONINJA_TEXT" x="3.81" y="-21.59" smashed="yes"/>
 </elements>
 <signals>
